File: 10AmpBuckV3.brd (EAGLE design)
At the start: 46.7 x 38.1 mm, 28 parts

Commit message: refining
Parts:
- removed 3V3REG: SPX3819M5-L-3-3, James:SOT95P280X145-5N
- removed C10: 10nf, SparkFun-Capacitors:0603-CAP
- removed C9: 4.7, SparkFun-Capacitors:1206
- added U$1: TPS75533, James:TO263-5
- C12, C8: device SparkFun-Capacitors:CPOL-RADIAL-10UF-25V -> SparkFun-Capacitors:CPOL-RADIAL-100UF-25V
- C7: value (none) -> 4.7; device SparkFun-Capacitors:CPOL-RADIAL-10UF-25V -> SparkFun-Capacitors:1206
- moved 3V3 8.89 mm to (43.2, 22.9)
- moved GND 7.73 mm to (44.5, 15.2), turned to 180 degrees
- moved C7 5.85 mm to (40.6, 14.0), flipped to the bottom, turned to 270 degrees
- moved C2 2.84 mm to (17.8, 12.7)
- moved ENABLE 2.84 mm to (3.81, 21.6)
- moved R2 2.54 mm to (8.89, 24.1)
- moved R3 2.54 mm to (8.89, 19.1)
- moved C12 1.27 mm to (12.7, 14.6)
- moved H2 1.27 mm to (6.35, 31.8)
Connections:
- removed net N$1: 3V3REG.4, C10.2
- net +3V3: now also C7.1, U$1.4; no longer 3V3REG.5
- net +5V: now also U$1.1, U$1.2; no longer 3V3REG.1, 3V3REG.3, C7.1, C9.1
- net GND: now also U$1.3, U$1.5, U$1.6; no longer 3V3REG.2, C10.1, C9.2
Routing:
- net +3V3: track 2.91 -> 15.8 mm
- net V+: track 10.4 -> 1.27 mm
- net N$1: track 5.17 -> 0.00 mm
- net ENABLE: track 25.8 -> 22.4 mm
- net GND: track 52.8 -> 55.9 mm, vias 33 -> 38
- net +5V: track 23.4 -> 21.0 mm
Other:
- board size 46.7 x 38.1 mm -> 46.7 x 36.9 mm
