File: 10AmpBuckV3.sch (EAGLE design)
At the start: 28 parts

Commit message: refining
Parts:
- removed 3V3REG: SPX3819M5-L-3-3, James:SPX3819M5-L-3-3
- removed C10: 10nf, SparkFun-Capacitors:CAP0603-CAP
- removed C9: 4.7, SparkFun-Capacitors:CAP1206
- added U$1: TPS75533, James:TPS75533
- C12, C8: device SparkFun-Capacitors:CAP_POLPTH2 -> SparkFun-Capacitors:CAP_POLPTH1
- C7: value (none) -> 4.7; device SparkFun-Capacitors:CAP_POLPTH2 -> SparkFun-Capacitors:CAP1206
Connections:
- removed net N$1: 3V3REG.ADJ/BYP, C10.2
- net +3V3: now also C7.1, U$1.OUT; no longer 3V3REG.VOUT
- net +5V: now also U$1.EN, U$1.IN; no longer 3V3REG.EN, 3V3REG.VIN, C7.+, C9.1
- net GND: now also C7.2, U$1.GND, U$1.GNDPAD, U$1.PG-BAR; no longer 3V3REG.GND, C10.1, C7.-, C9.2
Changed lines of the file:
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@@
 <part name="C6" library="SparkFun-Capacitors" deviceset="CAP" device="1206" value="10uf"/>
 <part name="GND6" library="supply1" deviceset="GND" device=""/>
-<part name="C7" library="SparkFun-Capacitors" deviceset="CAP_POL" device="PTH2"/>
-<part name="C8" library="SparkFun-Capacitors" deviceset="CAP_POL" device="PTH2"/>
+<part name="C8" library="SparkFun-Capacitors" deviceset="CAP_POL" device="PTH1"/>
 <part name="H2" library="holes" deviceset="MOUNT-PAD-ROUND" device="5.5" value="MOUNT-PAD-ROUND5.5"/>
 <part name="H1" library="holes" deviceset="MOUNT-PAD-ROUND" device="5.5" value="MOUNT-PAD-ROUND5.5"/>
 <part name="H3" library="holes" deviceset="MOUNT-PAD-ROUND" device="5.5" value="MOUNT-PAD-ROUND5.5"/>
 <part name="H4" library="holes" deviceset="MOUNT-PAD-ROUND" device="5.5" value="MOUNT-PAD-ROUND5.5"/>
-<part name="3V3REG" library="James" deviceset="SPX3819M5-L-3-3" device=""/>
-<part name="C9" library="SparkFun-Capacitors" deviceset="CAP" device="1206" value="4.7"/>
 <part name="P+2" library="supply1" deviceset="+5V" device=""/>
 <part name="GND3" library="supply1" deviceset="GND" device=""/>
@@
 <part name="3V3" library="wirepad" deviceset="WIREPAD" device="SMD2,54-5,08"/>
 <part name="GND" library="wirepad" deviceset="WIREPAD" device="SMD2,54-5,08"/>
-<part name="C10" library="SparkFun-Capacitors" deviceset="CAP" device="0603-CAP" value="10nf"/>
 <part name="R1" library="SparkFun-Passives" deviceset="RESISTOR" device="0603-RES"/>
 <part name="LED1" library="LilyPad-Wearables" deviceset="LED" device="1206"/>
 <part name="GND8" library="supply1" deviceset="GND" device=""/>
-<part name="C12" library="SparkFun-Capacitors" deviceset="CAP_POL" device="PTH2"/>
+<part name="C12" library="SparkFun-Capacitors" deviceset="CAP_POL" device="PTH1"/>
 <part name="C13" library="SparkFun-Capacitors" deviceset="CAP" device="1206" value="4.7"/>
 <part name="ENABLE" library="wirepad" deviceset="WIREPAD" device="SMD2,54-5,08"/>
@@
 <part name="SUPPLY2" library="supply2" deviceset="V+" device=""/>
 <part name="GND10" library="supply1" deviceset="GND" device=""/>
+<part name="U$1" library="James" deviceset="TPS75533" device=""/>
+<part name="GND11" library="supply1" deviceset="GND" device=""/>
+<part name="C7" library="SparkFun-Capacitors" deviceset="CAP" device="1206" value="4.7"/>
 </parts>
 <sheets>
@@
 <instance part="C6" gate="G$1" x="93.98" y="48.26"/>
 <instance part="GND6" gate="1" x="93.98" y="38.1"/>
-<instance part="C7" gate="G$1" x="99.06" y="50.8"/>
 <instance part="C8" gate="G$1" x="104.14" y="50.8"/>
 <instance part="H2" gate="G$1" x="-48.26" y="78.74" rot="R180"/>
@@
 <instance part="H3" gate="G$1" x="147.32" y="53.34"/>
 <instance part="H4" gate="G$1" x="2.54" y="50.8" rot="R180"/>
-<instance part="3V3REG" gate="A" x="99.06" y="111.76"/>
-<instance part="C9" gate="G$1" x="60.96" y="109.22"/>
 <instance part="P+2" gate="1" x="60.96" y="116.84"/>
 <instance part="GND3" gate="1" x="60.96" y="99.06"/>
@@
 <instance part="3V3" gate="G$1" x="147.32" y="119.38" rot="R180"/>
 <instance part="GND" gate="G$1" x="73.66" y="93.98"/>
-<instance part="C10" gate="G$1" x="71.12" y="109.22" rot="R180"/>
 <instance part="R1" gate="G$1" x="134.62" y="66.04" rot="R180"/>
 <instance part="LED1" gate="G$1" x="147.32" y="66.04" rot="R90"/>
@@
 <instance part="SUPPLY2" gate="1" x="22.86" y="129.54"/>
 <instance part="GND10" gate="1" x="7.62" y="55.88"/>
+<instance part="U$1" gate="G$1" x="99.06" y="132.08"/>
+<instance part="GND11" gate="1" x="127" y="101.6"/>
+<instance part="C7" gate="G$1" x="127" y="109.22"/>
 </instances>
 <busses>
@@
 <pinref part="GND7" gate="1" pin="GND"/>
 <wire x1="109.22" y1="43.18" x2="109.22" y2="40.64" width="0.1524" layer="91"/>
-<pinref part="C7" gate="G$1" pin="-"/>
-<wire x1="99.06" y1="45.72" x2="99.06" y2="40.64" width="0.1524" layer="91"/>
 <pinref part="C8" gate="G$1" pin="-"/>
-<wire x1="99.06" y1="40.64" x2="104.14" y2="40.64" width="0.1524" layer="91"/>
 <wire x1="104.14" y1="40.64" x2="104.14" y2="45.72" width="0.1524" layer="91"/>
 <wire x1="104.14" y1="40.64" x2="109.22" y2="40.64" width="0.1524" layer="91"/>
-<junction x="104.14" y="40.64"/>
 <junction x="109.22" y="40.64"/>
 <pinref part="C13" gate="G$1" pin="2"/>
@@
 </segment>
 <segment>
-<pinref part="3V3REG" gate="A" pin="GND"/>
-<pinref part="C9" gate="G$1" pin="2"/>
-<wire x1="81.28" y1="101.6" x2="71.12" y2="101.6" width="0.1524" layer="91"/>
-<wire x1="71.12" y1="101.6" x2="60.96" y2="101.6" width="0.1524" layer="91"/>
-<wire x1="60.96" y1="101.6" x2="60.96" y2="106.68" width="0.1524" layer="91"/>
+<wire x1="81.28" y1="101.6" x2="60.96" y2="101.6" width="0.1524" layer="91"/>
 <pinref part="GND3" gate="1" pin="GND"/>
-<junction x="60.96" y="101.6"/>
 <pinref part="GND" gate="G$1" pin="P"/>
 <wire x1="76.2" y1="93.98" x2="81.28" y2="93.98" width="0.1524" layer="91"/>
 <wire x1="81.28" y1="93.98" x2="81.28" y2="101.6" width="0.1524" layer="91"/>
+<pinref part="U$1" gate="G$1" pin="GND"/>
+<wire x1="96.52" y1="119.38" x2="96.52" y2="114.3" width="0.1524" layer="91"/>
+<wire x1="96.52" y1="114.3" x2="96.52" y2="101.6" width="0.1524" layer="91"/>
+<wire x1="96.52" y1="101.6" x2="81.28" y2="101.6" width="0.1524" layer="91"/>
 <junction x="81.28" y="101.6"/>
-<pinref part="C10" gate="G$1" pin="1"/>
-<wire x1="71.12" y1="104.14" x2="71.12" y2="101.6" width="0.1524" layer="91"/>
-<junction x="71.12" y="101.6"/>
+<pinref part="U$1" gate="G$1" pin="GNDPAD"/>
+<wire x1="96.52" y1="114.3" x2="99.06" y2="114.3" width="0.1524" layer="91"/>
+<wire x1="99.06" y1="114.3" x2="99.06" y2="119.38" width="0.1524" layer="91"/>
+<junction x="96.52" y="114.3"/>
+<pinref part="U$1" gate="G$1" pin="PG-BAR"/>
+<wire x1="104.14" y1="119.38" x2="109.22" y2="119.38" width="0.1524" layer="91"/>
+<wire x1="96.52" y1="101.6" x2="109.22" y2="101.6" width="0.1524" layer="91"/>
+<wire x1="109.22" y1="101.6" x2="109.22" y2="119.38" width="0.1524" layer="91"/>
+<junction x="96.52" y="101.6"/>
 </segment>
 <segment>
@@
 <pinref part="GND10" gate="1" pin="GND"/>
 <wire x1="12.7" y1="58.42" x2="7.62" y2="58.42" width="0.1524" layer="91"/>
+</segment>
+<segment>
+<pinref part="GND11" gate="1" pin="GND"/>
+<wire x1="127" y1="106.68" x2="127" y2="104.14" width="0.1524" layer="91"/>
+<pinref part="C7" gate="G$1" pin="2"/>
 </segment>
 </net>
@@
 <wire x1="91.44" y1="55.88" x2="93.98" y2="55.88" width="0.1524" layer="91"/>
 <junction x="91.44" y="55.88"/>
-<wire x1="93.98" y1="55.88" x2="99.06" y2="55.88" width="0.1524" layer="91"/>
-<wire x1="99.06" y1="55.88" x2="104.14" y2="55.88" width="0.1524" layer="91"/>
+<wire x1="93.98" y1="55.88" x2="104.14" y2="55.88" width="0.1524" layer="91"/>
 <wire x1="104.14" y1="55.88" x2="109.22" y2="55.88" width="0.1524" layer="91"/>
 <wire x1="91.44" y1="55.88" x2="88.9" y2="55.88" width="0.1524" layer="91"/>
@@
 <wire x1="93.98" y1="53.34" x2="93.98" y2="55.88" width="0.1524" layer="91"/>
 <junction x="93.98" y="55.88"/>
-<pinref part="C7" gate="G$1" pin="+"/>
-<wire x1="99.06" y1="55.88" x2="99.06" y2="53.34" width="0.1524" layer="91"/>
-<junction x="99.06" y="55.88"/>
 <pinref part="C8" gate="G$1" pin="+"/>
 <wire x1="104.14" y1="55.88" x2="104.14" y2="53.34" width="0.1524" layer="91"/>
@@
 </segment>
 <segment>
-<pinref part="3V3REG" gate="A" pin="VIN"/>
-<pinref part="C9" gate="G$1" pin="1"/>
-<wire x1="81.28" y1="114.3" x2="76.2" y2="114.3" width="0.1524" layer="91"/>
-<pinref part="3V3REG" gate="A" pin="EN"/>
 <wire x1="76.2" y1="114.3" x2="60.96" y2="114.3" width="0.1524" layer="91"/>
-<wire x1="81.28" y1="109.22" x2="76.2" y2="109.22" width="0.1524" layer="91"/>
 <wire x1="76.2" y1="109.22" x2="76.2" y2="114.3" width="0.1524" layer="91"/>
 <junction x="76.2" y="114.3"/>
 <pinref part="P+2" gate="1" pin="+5V"/>
-<junction x="60.96" y="114.3"/>
+<pinref part="U$1" gate="G$1" pin="EN"/>
+<wire x1="76.2" y1="114.3" x2="91.44" y2="114.3" width="0.1524" layer="91"/>
+<wire x1="91.44" y1="114.3" x2="91.44" y2="119.38" width="0.1524" layer="91"/>
+<pinref part="U$1" gate="G$1" pin="IN"/>
+<wire x1="76.2" y1="109.22" x2="93.98" y2="109.22" width="0.1524" layer="91"/>
+<wire x1="93.98" y1="109.22" x2="93.98" y2="119.38" width="0.1524" layer="91"/>
 </segment>
 </net>
@@
 <net name="+3V3" class="0">
 <segment>
-<pinref part="3V3REG" gate="A" pin="VOUT"/>
-<wire x1="116.84" y1="114.3" x2="132.08" y2="114.3" width="0.1524" layer="91"/>
 <pinref part="+3V1" gate="G$1" pin="+3V3"/>
 <wire x1="134.62" y1="121.92" x2="132.08" y2="121.92" width="0.1524" layer="91"/>
@@
 <junction x="132.08" y="119.38"/>
 <pinref part="3V3" gate="G$1" pin="P"/>
-</segment>
-</net>
-<net name="N$1" class="0">
-<segment>
-<pinref part="3V3REG" gate="A" pin="ADJ/BYP"/>
-<wire x1="81.28" y1="106.68" x2="73.66" y2="106.68" width="0.1524" layer="91"/>
-<wire x1="73.66" y1="106.68" x2="73.66" y2="111.76" width="0.1524" layer="91"/>
-<pinref part="C10" gate="G$1" pin="2"/>
-<wire x1="73.66" y1="111.76" x2="71.12" y2="111.76" width="0.1524" layer="91"/>
-</segment>
-</net>
+<pinref part="U$1" gate="G$1" pin="OUT"/>
+<wire x1="101.6" y1="119.38" x2="101.6" y2="114.3" width="0.1524" layer="91"/>
+<wire x1="101.6" y1="114.3" x2="127" y2="114.3" width="0.1524" layer="91"/>
+<pinref part="C7" gate="G$1" pin="1"/>
+<wire x1="127" y1="114.3" x2="132.08" y2="114.3" width="0.1524" layer="91"/>
+<junction x="127" y="114.3"/>
+</segment>
+</net>
